File: eagle/AD9833_FG/AD9833_FG_Main.sch (EAGLE design)
At the start: 27 parts, among them IC1 ATMEGA48/88/168, IC2 AD9833_MODULE, IC3 NJM2396, IC4 HT7330, Q1 16MHz, X1 OUT, X2 PWR

Commit message: Update eagle files
Parts:
- removed X1: OUT, con-wago-508:W237-02P
- removed X2: PWR, con-wago-508:W237-02P
- added SL1: OUT, con-amp-quick:M02
- added SL2: PWR, con-amp-quick:M02
Connections:
- net GND: no longer X1-2.KL, X2-2.KL
- net N$15: now also SL2.2; no longer X2-1.KL
- net N$6: now also SL1.2; no longer X1-1.KL
Changed lines of the file:
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@@
 <setting verticaltext="up"/>
 </settings>
-<grid distance="0.1" unitdist="inch" unit="inch" style="lines" multiple="1" display="yes" altdistance="0.01" altunitdist="inch" altunit="inch"/>
+<grid distance="0.1" unitdist="inch" unit="inch" style="lines" multiple="1" display="no" altdistance="0.01" altunitdist="inch" altunit="inch"/>
 <layers>
 <layer number="1" name="Top" color="4" fill="1" visible="no" active="no"/>
@@
 <part name="JP6" library="pinhead" deviceset="PINHD-1X2" device="" value="TP_GND"/>
 <part name="GND16" library="supply1" deviceset="GND" device=""/>
-<part name="X1" library="con-wago-508" deviceset="W237-02P" device="" value="OUT"/>
-<part name="X2" library="con-wago-508" deviceset="W237-02P" device="" value="PWR"/>
 <part name="P+5" library="supply1" deviceset="+5V" device=""/>
 <part name="R6" library="rcl" deviceset="R-EU_" device="0207/7" value="1k"/>
@@
 <part name="C8" library="rcl" deviceset="C-EU" device="025-024X044" value="0.1uF"/>
 <part name="P+7" library="supply1" deviceset="+5V" device=""/>
+<part name="SL1" library="con-amp-quick" deviceset="M02" device="" value="OUT"/>
+<part name="SL2" library="con-amp-quick" deviceset="M02" device="" value="PWR"/>
 </parts>
 <sheets>
@@
 <instance part="JP6" gate="G$1" x="22.86" y="139.7" rot="MR0"/>
 <instance part="GND16" gate="1" x="33.02" y="132.08"/>
-<instance part="X1" gate="-1" x="73.66" y="124.46" smashed="yes">
-<attribute name="NAME" x="72.39" y="125.349" size="1.778" layer="95" rot="R180"/>
-</instance>
-<instance part="X1" gate="-2" x="73.66" y="119.38" smashed="yes">
-<attribute name="VALUE" x="68.58" y="127" size="1.778" layer="96"/>
-<attribute name="NAME" x="72.39" y="120.269" size="1.778" layer="95" rot="R180"/>
-</instance>
-<instance part="X2" gate="-1" x="22.86" y="73.66" smashed="yes">
-<attribute name="NAME" x="21.59" y="74.549" size="1.778" layer="95" rot="R180"/>
-</instance>
-<instance part="X2" gate="-2" x="22.86" y="68.58" smashed="yes">
-<attribute name="VALUE" x="17.78" y="76.2" size="1.778" layer="96"/>
-<attribute name="NAME" x="21.59" y="69.469" size="1.778" layer="95" rot="R180"/>
-</instance>
 <instance part="P+5" gate="1" x="45.72" y="154.94"/>
 <instance part="R6" gate="G$1" x="45.72" y="144.78" rot="R90"/>
@@
 <instance part="C8" gate="G$1" x="210.82" y="119.38" rot="R90"/>
 <instance part="P+7" gate="1" x="218.44" y="137.16" rot="MR0"/>
+<instance part="SL1" gate="G$1" x="71.12" y="121.92"/>
+<instance part="SL2" gate="G$1" x="20.32" y="71.12"/>
 </instances>
 <busses>
@@
 </segment>
 <segment>
-<wire x1="78.74" y1="119.38" x2="86.36" y2="119.38" width="0.1524" layer="91"/>
-<wire x1="86.36" y1="119.38" x2="86.36" y2="106.68" width="0.1524" layer="91"/>
+<wire x1="78.74" y1="121.92" x2="86.36" y2="121.92" width="0.1524" layer="91"/>
+<wire x1="86.36" y1="121.92" x2="86.36" y2="106.68" width="0.1524" layer="91"/>
 <pinref part="GND2" gate="1" pin="GND"/>
-<pinref part="X1" gate="-2" pin="KL"/>
 </segment>
 <segment>
@@
 </segment>
 <segment>
-<wire x1="27.94" y1="68.58" x2="30.48" y2="68.58" width="0.1524" layer="91"/>
+<wire x1="27.94" y1="71.12" x2="30.48" y2="71.12" width="0.1524" layer="91"/>
 <pinref part="GND7" gate="1" pin="GND"/>
-<wire x1="30.48" y1="68.58" x2="30.48" y2="43.18" width="0.1524" layer="91"/>
-<pinref part="X2" gate="-2" pin="KL"/>
+<wire x1="30.48" y1="71.12" x2="30.48" y2="43.18" width="0.1524" layer="91"/>
 </segment>
 <segment>
@@
 <pinref part="IC2" gate="G$1" pin="OUT"/>
 <wire x1="86.36" y1="137.16" x2="81.28" y2="137.16" width="0.1524" layer="91"/>
-<pinref part="X1" gate="-1" pin="KL"/>
+<pinref part="SL1" gate="G$1" pin="2"/>
 </segment>
 </net>
@@
 <wire x1="40.64" y1="71.12" x2="40.64" y2="73.66" width="0.1524" layer="91"/>
 <junction x="40.64" y="73.66"/>
-<pinref part="X2" gate="-1" pin="KL"/>
-</segment>
-</net>
+<pinref part="SL2" gate="G$1" pin="2"/>
+</segment>
+</net>
