File: eagle/AD9833_FG/AD9833_FG_Out.sch (EAGLE design)
At the start: 12 parts, among them IC1 AD822N

Commit message: Board Design
Parts:
- removed JP1: IN, pinhead:PINHD-1X2
- removed JP2: OUT, pinhead:PINHD-1X2
- removed JP3, JP5: PWR, pinhead:PINHD-1X2
- added SL1: IN, con-amp-quick:M02
- added SL2: OUT, con-amp-quick:M02
- added SL3, SL4: PWR, con-amp-quick:M02
- R1: value 4.7k -> 8.2k
- R2: value 12k -> 1k
Connections:
- removed net N$3: IC1A.IN+, JP1.1
- new net N$2: IC1A.IN+, SL1.1
- net AGND: now also SL1.2, SL2.1, SL3.1, SL4.2; no longer JP1.2, JP2.2, JP3.2, JP5.2
- net N$5: now also SL2.2; no longer JP2.1
- net V+: now also SL3.2, SL4.1; no longer JP3.1, JP5.1
Other:
- moved on the sheet: C1, C2, IC1A, IC1B, IC1P, JP4, LED1, R1, R2, R3

Commit message: Update eagle files
Parts:
- removed SL4: PWR, con-amp-quick:M02
- R3: value 4.7k -> 2.2k
- SL3: device con-amp-quick:M02 -> con-amp-quick:M04
Connections:
- net AGND: now also SL2.2, SL3.2, SL3.3; no longer SL2.1, SL3.1, SL4.2
- net N$5: now also SL2.1; no longer SL2.2
- net V+: now also SL3.1, SL3.4; no longer SL3.2, SL4.1
Other:
- moved on the sheet: SL2
Changed lines of the file:
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@@
 <setting verticaltext="up"/>
 </settings>
-<grid distance="0.1" unitdist="inch" unit="inch" style="lines" multiple="1" display="yes" altdistance="0.01" altunitdist="inch" altunit="inch"/>
+<grid distance="0.1" unitdist="inch" unit="inch" style="lines" multiple="1" display="no" altdistance="0.01" altunitdist="inch" altunit="inch"/>
 <layers>
 <layer number="1" name="Top" color="4" fill="1" visible="no" active="no"/>
@@
 <part name="AGND6" library="supply1" deviceset="AGND" device=""/>
 <part name="LED1" library="led" deviceset="LED" device="3MM" value="GREEN"/>
-<part name="R3" library="rcl" deviceset="R-EU_" device="0207/7" value="4.7k"/>
+<part name="R3" library="rcl" deviceset="R-EU_" device="0207/7" value="2.2k"/>
 <part name="P+3" library="supply1" deviceset="V+" device=""/>
 <part name="AGND7" library="supply1" deviceset="AGND" device=""/>
@@
 <part name="SL1" library="con-amp-quick" deviceset="M02" device="" value="IN"/>
 <part name="SL2" library="con-amp-quick" deviceset="M02" device="" value="OUT"/>
-<part name="SL3" library="con-amp-quick" deviceset="M02" device="" value="PWR"/>
-<part name="SL4" library="con-amp-quick" deviceset="M02" device="" value="PWR"/>
+<part name="SL3" library="con-amp-quick" deviceset="M04" device="" value="PWR"/>
 </parts>
 <sheets>
@@
 <instance part="FRAME1" gate="G$1" x="0" y="0"/>
 <instance part="SL1" gate="G$1" x="73.66" y="83.82" rot="MR180"/>
-<instance part="SL2" gate="G$1" x="172.72" y="76.2" rot="MR0"/>
-<instance part="SL3" gate="G$1" x="73.66" y="119.38"/>
-<instance part="SL4" gate="G$1" x="73.66" y="134.62"/>
+<instance part="SL2" gate="G$1" x="172.72" y="78.74" rot="R180"/>
+<instance part="SL3" gate="G$1" x="76.2" y="116.84"/>
 </instances>
 <busses>
@@
 </segment>
 <segment>
-<wire x1="165.1" y1="76.2" x2="160.02" y2="76.2" width="0.1524" layer="91"/>
 <wire x1="160.02" y1="76.2" x2="160.02" y2="63.5" width="0.1524" layer="91"/>
 <pinref part="AGND2" gate="VR1" pin="AGND"/>
-<pinref part="SL2" gate="G$1" pin="1"/>
+<pinref part="SL2" gate="G$1" pin="2"/>
+<wire x1="160.02" y1="76.2" x2="165.1" y2="76.2" width="0.1524" layer="91"/>
 </segment>
 <segment>
 <pinref part="AGND3" gate="VR1" pin="AGND"/>
-<wire x1="88.9" y1="106.68" x2="88.9" y2="119.38" width="0.1524" layer="91"/>
+<wire x1="88.9" y1="119.38" x2="88.9" y2="116.84" width="0.1524" layer="91"/>
+<wire x1="88.9" y1="116.84" x2="88.9" y2="106.68" width="0.1524" layer="91"/>
 <wire x1="81.28" y1="119.38" x2="88.9" y2="119.38" width="0.1524" layer="91"/>
-<pinref part="SL3" gate="G$1" pin="1"/>
-<wire x1="81.28" y1="137.16" x2="88.9" y2="137.16" width="0.1524" layer="91"/>
-<pinref part="SL4" gate="G$1" pin="2"/>
-<wire x1="88.9" y1="137.16" x2="88.9" y2="119.38" width="0.1524" layer="91"/>
-<junction x="88.9" y="119.38"/>
+<pinref part="SL3" gate="G$1" pin="3"/>
+<pinref part="SL3" gate="G$1" pin="2"/>
+<wire x1="81.28" y1="116.84" x2="88.9" y2="116.84" width="0.1524" layer="91"/>
+<junction x="88.9" y="116.84"/>
 </segment>
 <segment>
@@
 <pinref part="IC1" gate="B" pin="OUT"/>
 <wire x1="152.4" y1="78.74" x2="149.86" y2="78.74" width="0.1524" layer="91"/>
+<pinref part="SL2" gate="G$1" pin="1"/>
 <wire x1="152.4" y1="78.74" x2="165.1" y2="78.74" width="0.1524" layer="91"/>
 <junction x="152.4" y="78.74"/>
-<pinref part="SL2" gate="G$1" pin="2"/>
 </segment>
 </net>
@@
 <wire x1="109.22" y1="121.92" x2="109.22" y2="124.46" width="0.1524" layer="91"/>
 <junction x="109.22" y="121.92"/>
-<pinref part="SL3" gate="G$1" pin="2"/>
-<wire x1="81.28" y1="134.62" x2="83.82" y2="134.62" width="0.1524" layer="91"/>
-<pinref part="SL4" gate="G$1" pin="1"/>
-<wire x1="83.82" y1="134.62" x2="83.82" y2="121.92" width="0.1524" layer="91"/>
+<pinref part="SL3" gate="G$1" pin="4"/>
+<pinref part="SL3" gate="G$1" pin="1"/>
+<wire x1="81.28" y1="114.3" x2="83.82" y2="114.3" width="0.1524" layer="91"/>
+<wire x1="83.82" y1="114.3" x2="83.82" y2="121.92" width="0.1524" layer="91"/>
 <junction x="83.82" y="121.92"/>
 </segment>

Commit message: Impl. Amp Board
Connections:
- net AGND: now also SL2.1; no longer SL2.2
- net N$5: now also SL2.2; no longer SL2.1
Other:
- moved on the sheet: SL2
Changed lines of the file:
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@@
 <instance part="FRAME1" gate="G$1" x="0" y="0"/>
 <instance part="SL1" gate="G$1" x="73.66" y="83.82" rot="MR180"/>
-<instance part="SL2" gate="G$1" x="172.72" y="78.74" rot="R180"/>
+<instance part="SL2" gate="G$1" x="172.72" y="76.2" rot="MR0"/>
 <instance part="SL3" gate="G$1" x="76.2" y="116.84"/>
 </instances>
@@
 <wire x1="160.02" y1="76.2" x2="160.02" y2="63.5" width="0.1524" layer="91"/>
 <pinref part="AGND2" gate="VR1" pin="AGND"/>
-<pinref part="SL2" gate="G$1" pin="2"/>
+<pinref part="SL2" gate="G$1" pin="1"/>
 <wire x1="160.02" y1="76.2" x2="165.1" y2="76.2" width="0.1524" layer="91"/>
 </segment>
@@
 <pinref part="IC1" gate="B" pin="OUT"/>
 <wire x1="152.4" y1="78.74" x2="149.86" y2="78.74" width="0.1524" layer="91"/>
-<pinref part="SL2" gate="G$1" pin="1"/>
+<pinref part="SL2" gate="G$1" pin="2"/>
 <wire x1="152.4" y1="78.74" x2="165.1" y2="78.74" width="0.1524" layer="91"/>
 <junction x="152.4" y="78.74"/>
