File: eagle/AD9833_FG/AD9833_FG_Main_3V3.brd (EAGLE design)
At the start: 53 x 63.5 mm, 19 parts, among them IC1 ATMEGA48/88/168, IC2 AD9833_MODULE, IC3 TA48M033F

Commit message: Update eagle files
Parts:
- removed R3: 3.3k, rcl:0207/7
- removed SL3: PWR, con-amp-quick:02P
- added JP3: TP_3V3, pinhead:1X02
- added R4: 100k, pot:B25P
- C5: device rcl:SANYO-OSCON_C -> rcl:E2,5-7
- C8: device rcl:C025-024X044 -> rcl:C050-024X044
- R2: value 12k -> 220k
- moved R2 42.6 mm to (6.35, 7.62), turned to 0 degrees
- moved JP6 41.0 mm to (45.7, 6.35), turned to 270 degrees
- moved R1 9.16 mm to (34.3, 63.5), turned to 180 degrees
- moved LCD1 8.03 mm to (21.6, 61.0)
- moved SL1 5.68 mm to (39.4, 7.62)
- moved IC1 5.68 mm to (22.9, 47.0)
- moved JP1 5.68 mm to (17.8, 30.5)
- moved JP2 5.68 mm to (21.6, 35.6)
- moved C7 5.68 mm to (24.1, 40.6)
- moved IC2 5.68 mm to (35.6, 17.8)
- moved C2 5.68 mm to (29.2, 7.62)
- moved R7 5.68 mm to (7.62, 36.8)
- moved C8 5.24 mm to (25.4, 53.3)
- moved C5 5.08 mm to (16.5, 17.8), turned to 180 degrees
- moved C1 5.08 mm to (14.0, 25.4)
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Connections:
- new net N$11: R2.1, R4.E
- net +3V3: now also JP3.1, JP3.2
- net GND: now also R4.A; no longer R3.1, SL3.1
- net N$15: no longer SL3.2
- net N$16: now also R4.S; no longer R2.1, R3.2
Routing:
- net +3V3: track 0.00 -> 193.7 mm, vias 0 -> 4
- net GND: track 0.00 -> 181.4 mm
- net N$2: track 0.00 -> 76.1 mm, vias 0 -> 4
- net N$1: track 0.00 -> 65.6 mm, vias 0 -> 2
- net N$16: track 0.00 -> 64.6 mm, vias 0 -> 2
- net N$3: track 0.00 -> 47.8 mm
- net N$4: track 0.00 -> 33.0 mm, vias 0 -> 2
- net N$7: track 0.00 -> 30.5 mm, vias 0 -> 2
- net N$5: track 0.00 -> 27.9 mm, vias 0 -> 2
- net N$15: track 0.00 -> 20.3 mm
- net N$9: track 0.00 -> 12.7 mm
- net N$8: track 0.00 -> 12.7 mm
- net N$14: track 0.00 -> 7.62 mm
- net N$6: track 0.00 -> 7.62 mm
- net N$10: track 0.00 -> 7.62 mm
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Other:
- board size 53 x 63.5 mm -> 47.9 x 73.7 mm

Commit message: Impl. Amp Board
Parts:
- moved JP6 22.9 mm to (22.9, 6.35)
Routing:
- net GND: track 181.4 -> 173.8 mm
- net N$2: track 76.1 -> 70.4 mm
Changed lines of the file:
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@@
 <element name="JP1" library="pinhead" package="1X03" value="RE" x="17.78" y="30.48"/>
 <element name="JP2" library="pinhead" package="1X02" value="SW" x="21.59" y="35.56"/>
-<element name="JP6" library="pinhead" package="1X02" value="TP_GND" x="45.72" y="6.35" rot="R270"/>
+<element name="JP6" library="pinhead" package="1X02" value="TP_GND" x="22.86" y="6.35" rot="R270"/>
 <element name="LCD1" library="mylib2" package="ATD_SPLC792-I2C" value="ATD_SPLC792-I2C" x="21.59" y="60.96"/>
 <element name="R1" library="rcl" package="0207/7" value="220" x="34.29" y="63.5" rot="R180"/>
@@
 <contactref element="IC2" pad="P$5"/>
 <wire x1="30.48" y1="50.8" x2="30.48" y2="53.34" width="0.4064" layer="16"/>
-<wire x1="46.99" y1="39.37" x2="43.18" y2="35.56" width="0.4064" layer="1"/>
+<wire x1="44.45" y1="36.83" x2="43.18" y2="35.56" width="0.4064" layer="1"/>
 <wire x1="43.18" y1="35.56" x2="43.18" y2="12.7" width="0.4064" layer="16"/>
 <wire x1="43.18" y1="12.7" x2="35.56" y2="12.7" width="0.4064" layer="1"/>
@@
 <via x="30.48" y="53.34" extent="1-16" drill="0.6" shape="square"/>
 <via x="43.18" y="35.56" extent="1-16" drill="0.6" shape="square"/>
-<wire x1="30.48" y1="53.34" x2="34.29" y2="57.15" width="0.4064" layer="1"/>
-<wire x1="34.29" y1="57.15" x2="45.72" y2="57.15" width="0.4064" layer="1"/>
-<wire x1="45.72" y1="57.15" x2="46.99" y2="55.88" width="0.4064" layer="1"/>
-<wire x1="46.99" y1="55.88" x2="46.99" y2="39.37" width="0.4064" layer="1"/>
+<wire x1="30.48" y1="53.34" x2="30.48" y2="54.61" width="0.4064" layer="1"/>
+<wire x1="30.48" y1="54.61" x2="44.45" y2="54.61" width="0.4064" layer="1"/>
+<wire x1="44.45" y1="54.61" x2="44.45" y2="36.83" width="0.4064" layer="1"/>
 <via x="43.18" y="12.7" extent="1-16" drill="0.6" shape="square"/>
 <via x="35.56" y="12.7" extent="1-16" drill="0.6" shape="square"/>
@@
 <wire x1="15.24" y1="22.86" x2="15.24" y2="17.78" width="1.016" layer="16"/>
 <wire x1="30.48" y1="7.62" x2="30.46" y2="7.62" width="1.016" layer="16"/>
-<wire x1="45.72" y1="5.08" x2="38.1" y2="5.08" width="1.016" layer="16"/>
-<wire x1="38.1" y1="5.08" x2="38.1" y2="7.62" width="1.016" layer="16"/>
-<wire x1="45.72" y1="7.62" x2="45.72" y2="5.08" width="1.016" layer="16"/>
+<wire x1="22.86" y1="7.62" x2="22.86" y2="5.08" width="1.016" layer="16"/>
 <wire x1="7.62" y1="12.7" x2="7.62" y2="5.08" width="1.016" layer="16"/>
-<wire x1="7.62" y1="5.08" x2="15.24" y2="5.08" width="1.016" layer="16"/>
 <wire x1="15.24" y1="5.08" x2="15.24" y2="7.62" width="1.016" layer="16"/>
 <wire x1="15.24" y1="25.4" x2="15.24" y2="7.62" width="1.016" layer="16"/>
-<wire x1="38.1" y1="5.08" x2="30.48" y2="5.08" width="1.016" layer="16"/>
-<wire x1="30.48" y1="5.08" x2="15.24" y2="5.08" width="1.016" layer="16"/>
-<wire x1="30.48" y1="7.62" x2="30.48" y2="5.08" width="1.016" layer="16"/>
 <wire x1="30.48" y1="15.24" x2="30.48" y2="7.64" width="1.016" layer="16"/>
 <wire x1="30.48" y1="7.64" x2="30.46" y2="7.62" width="1.016" layer="16"/>
@@
 <wire x1="30.48" y1="40.64" x2="30.48" y2="15.24" width="1.016" layer="16"/>
 <wire x1="25.4" y1="43.18" x2="25.4" y2="40.64" width="1.016" layer="16"/>
+<wire x1="15.24" y1="5.08" x2="22.86" y2="5.08" width="1.016" layer="16"/>
+<wire x1="30.48" y1="7.64" x2="30.48" y2="5.08" width="1.016" layer="16"/>
+<wire x1="30.48" y1="5.08" x2="22.86" y2="5.08" width="1.016" layer="16"/>
+<wire x1="38.1" y1="7.62" x2="38.1" y2="5.08" width="1.016" layer="16"/>
+<wire x1="38.1" y1="5.08" x2="30.48" y2="5.08" width="1.016" layer="16"/>
+<wire x1="7.62" y1="5.08" x2="15.24" y2="5.08" width="1.016" layer="16"/>
 </signal>
 <signal name="N$6">

Commit message: Update
Parts:
- IC1: value ATMEGA48/88/168 -> ATMEGA328P
Changed lines of the file:
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@@
 <element name="C7" library="rcl" package="C025-024X044" value="0.1uF" x="24.13" y="40.64" rot="R180"/>
 <element name="C8" library="rcl" package="C050-024X044" value="0.1uF" x="25.4" y="53.34"/>
-<element name="IC1" library="mylib2" package="DIL28-3" value="ATMEGA48/88/168" x="22.86" y="46.99"/>
+<element name="IC1" library="mylib2" package="DIL28-3" value="ATMEGA328P" x="22.86" y="46.99"/>
 <element name="IC2" library="mylib2" package="AD9833_MODULE" value="AD9833_MODULE" x="35.56" y="17.78"/>
 <element name="IC3" library="mylib2" package="TA48MXXX" value="TA48M033F" x="15.24" y="22.86"/>
